Commit message: Correction sur le pointage quand pt non atteignable

File: structure_lego.urdf (robot description, URDF)
Before this commit: robot structure_lego, 6 links, 5 joints
Links:
- link Outil: mass None -> 0.011
- link link1: mass None -> 0.572
- link link2: mass None -> 0.096
- link link3: mass None -> 0.097
